Commit message: add package keyboard in ros 1.0.7 Merge pull request #13 from asukiaaa/patch-3
Add rosrun command to specify values

File: mybot_description/urdf/mybot.xacro (robot description, xacro)
@@ -3,4 +3,9 @@
     <xacro:property name="cameraSize" value="0.05"/>
     <xacro:property name="cameraMass" value="0.1"/>
+    <xacro:include filename="$(find mybot_description)/urdf/mybot.gazebo" />
+    <!--<xacro:include filename="$(find mybot_description)/urdf/_d435.urdf.xacro"/>-->
+     <!--<sensor_d435 parent="base_footprint">-->
+        <!--<origin xyz="0 0 0" rpy="0 0 0"/>-->
+      <!--</sensor_d435>-->
     <!--base_footprint-->
     <link name="base_footprint">
@@ -56,4 +61,7 @@
                 <mesh filename="package://mybot_description/meshes/wheel.STL"/>
             </geometry>
+            <material name="black">
+                <color rgba="0.0 0.0 0.0 1"/>
+            </material>
         </visual>
         <inertial>
@@ -79,4 +87,7 @@
                 <mesh filename="package://mybot_description/meshes/wheel.STL"/>
             </geometry>
+            <material name="black">
+                <color rgba="0.0 0.0 0.0 1"/>
+            </material>
         </visual>
         <inertial>
